File: Satisfactron_2025.kicad_pcb (KiCad board)
At the start: 2 copper layers, 100 x 77 mm, 116 parts, among them J1 Conn_01x03, J10 Conn_01x04, J11 Conn_01x03, J12 Conn_01x03, J13 Conn_01x03, J14 Conn_01x03, J15 Conn_01x02, J16 Conn_01x04, J17 Conn_01x02, J18 Conn_01x02, J19 Conn_01x02, J2 Conn_01x08, J20 Conn_01x03, J3 Conn_01x02, J4 65100516121, J5 Conn_01x05, J6 Conn_01x06, J7 Conn_01x02, J8 Conn_01x04, J9 Conn_01x04, Q1 G2302, Q2 G2302, SW1 SW_DPST_x2, SW2 SW_Push, SW3 SW_Push, SW4 SW_Push, SW5 SW_Push, SW6 SW_Push, SW7 SW_Push, U1 AMS1117-3.3, U2 Adafruit BNO085, U3 ESP32-S3-WROOM-1-N16R8, U4 TMC2226, U5 TMC2226

Commit message: Add DXF, sch placement + start PCB placement
Parts:
- removed C1, C16, C19, C20, C21, C3, C5, C6: 100nF, Capacitor_SMD:C_0603_1608Metric_Pad1.08x0.95mm_HandSolder
- removed C24: 10uF, Capacitor_SMD:C_0805_2012Metric
- removed G*** (x2): LOGO, LOGO
- removed J10, J9: Conn_01x04, Connector_PinHeader_2.54mm:PinHeader_1x04_P2.54mm_Horizontal
- removed J12, J13, J14, J20: Conn_01x03, Connector_PinHeader_2.54mm:PinHeader_1x03_P2.54mm_Vertical
- removed J15, J7: Conn_01x02, Connector_Wire:SolderWire-0.75sqmm_1x02_P4.8mm_D1.25mm_OD2.3mm
- removed J16: Conn_01x04, Connector_PinHeader_2.54mm:PinHeader_1x04_P2.54mm_Vertical
- removed J17, J18, J19: Conn_01x02, Connector_PinHeader_2.54mm:PinHeader_1x02_P2.54mm_Vertical
- removed J8: Conn_01x04, Carte_Mere_PAMI_2025:Ecran_OLED0.9_Waveshare
- removed JP1: ID1, Jumper:SolderJumper-2_P1.3mm_Open_RoundedPad1.0x1.5mm
- removed JP10, JP8: SolderJumper_2_Bridged, Resistor_SMD:R_0402_1005Metric
- removed JP11, JP9: SolderJumper_2_Bridged, Carte_Mere_PAMI_2025:R_0402_1005Metric_jumperClosed
- removed JP2, JP4: MS2, Jumper:SolderJumper-2_P1.3mm_Open_RoundedPad1.0x1.5mm
- removed JP3, JP5: MS1, Jumper:SolderJumper-2_P1.3mm_Open_RoundedPad1.0x1.5mm
- removed Q1: G2302, Package_TO_SOT_SMD:SOT-23
- removed R1, R8: 1k, Resistor_SMD:R_0603_1608Metric_Pad0.98x0.95mm_HandSolder
- removed R2, R3, R6, R7: 10K, Resistor_SMD:R_0603_1608Metric_Pad0.98x0.95mm_HandSolder
- removed R21, R22, R5: 10k, Resistor_SMD:R_0603_1608Metric_Pad0.98x0.95mm_HandSolder
- removed R4: 68, Resistor_SMD:R_0603_1608Metric_Pad0.98x0.95mm_HandSolder
- removed U2: Adafruit BNO085, ComponentsEvo:Adafruit BNO085
- added C30: 22uF, Capacitor_SMD:C_0805_2012Metric, F.Cu at (493.2, 85.3)
- added D11: XL-3210RGBC-YG, LED_KSL:LED-ARRAY-SMD_HS-1204-RGB, F.Cu at (476.8, 126.0)
- added D12: XL-3210RGBC-YG, LED_KSL:LED-ARRAY-SMD_HS-1204-RGB, F.Cu at (476.8, 128.9)
- added D13: XL-3210RGBC-YG, LED_KSL:LED-ARRAY-SMD_HS-1204-RGB, F.Cu at (476.8, 131.8)
- added D14: XL-3210RGBC-YG, LED_KSL:LED-ARRAY-SMD_HS-1204-RGB, F.Cu at (476.8, 134.8)
- added D4: XL-3210RGBC-YG, LED_KSL:LED-ARRAY-SMD_HS-1204-RGB, F.Cu at (472.1, 128.9)
- added H10: SMTSO3040CTJ, Fastener_KSL:SMD-1_BD5.5-D4.0, F.Cu at (438.1, 90.9)
- added H11: SMTSO3040CTJ, Fastener_KSL:SMD-1_BD5.5-D4.0, F.Cu at (445.8, 75.6)
- added H12: SMTSO3040CTJ, Fastener_KSL:SMD-1_BD5.5-D4.0, F.Cu at (445.8, 83.2)
- added H13: SMTSO3040CTJ, Fastener_KSL:SMD-1_BD5.5-D4.0, F.Cu at (445.8, 90.9)
- added H14: SMTSO3040CTJ, Fastener_KSL:SMD-1_BD5.5-D4.0, F.Cu at (453.5, 75.6)
- added H15: SMTSO3040CTJ, Fastener_KSL:SMD-1_BD5.5-D4.0, F.Cu at (453.5, 83.2)
- added H16: SMTSO3040CTJ, Fastener_KSL:SMD-1_BD5.5-D4.0, F.Cu at (453.5, 90.9)
- added H17: SMTSO3040CTJ, Fastener_KSL:SMD-1_BD5.5-D4.0, F.Cu at (461.1, 75.6)
- added H18: SMTSO3040CTJ, Fastener_KSL:SMD-1_BD5.5-D4.0, F.Cu at (461.1, 83.2)
- added H19: SMTSO3040CTJ, Fastener_KSL:SMD-1_BD5.5-D4.0, F.Cu at (461.1, 90.9)
- added H5: SMTSO3040CTJ, Fastener_KSL:SMD-1_BD5.5-D4.0, F.Cu at (430.5, 75.6)
- added H6: SMTSO3040CTJ, Fastener_KSL:SMD-1_BD5.5-D4.0, F.Cu at (430.5, 83.2)
- added H7: SMTSO3040CTJ, Fastener_KSL:SMD-1_BD5.5-D4.0, F.Cu at (430.5, 90.9)
- added H8: SMTSO3040CTJ, Fastener_KSL:SMD-1_BD5.5-D4.0, F.Cu at (438.1, 75.6)
- added H9: SMTSO3040CTJ, Fastener_KSL:SMD-1_BD5.5-D4.0, F.Cu at (438.1, 83.2)
- added R27: 10k, Resistor_SMD:R_0603_1608Metric, F.Cu at (484.3, 78.0)
- added R28: 100k, Resistor_SMD:R_0603_1608Metric, F.Cu at (484.3, 80.5)
- added R29: 510k, Resistor_SMD:R_0603_1608Metric, F.Cu at (484.3, 83.0)
- added R30: 13k, Resistor_SMD:R_0603_1608Metric, F.Cu at (484.3, 85.5)
- added R31: 100k, Resistor_SMD:R_0603_1608Metric, F.Cu at (484.3, 88.1)
- added R32: 4.7k, Resistor_SMD:R_0603_1608Metric, F.Cu at (484.3, 90.6)
- added SW10: SPVN310101, Switch_KSL:SW-SMD_SPVN310101, F.Cu at (495.3, 108.5)
- added SW11: TS-1088-AR02016, Switch_KSL:SW-SMD_L3.9-W3.0-P4.45, F.Cu at (490.4, 126.0)
- added SW12: TS-1088-AR02016, Switch_KSL:SW-SMD_L3.9-W3.0-P4.45, F.Cu at (490.4, 130.3)
- added SW13: TS-1088-AR02016, Switch_KSL:SW-SMD_L3.9-W3.0-P4.45, F.Cu at (490.4, 134.5)
- added SW14: TS-1088-AR02016, Switch_KSL:SW-SMD_L3.9-W3.0-P4.45, F.Cu at (490.4, 138.7)
- added SW8: SPVN310101, Switch_KSL:SW-SMD_SPVN310101, F.Cu at (483.9, 108.5)
- added SW9: SPVN310101, Switch_KSL:SW-SMD_SPVN310101, F.Cu at (489.6, 108.5)
- added U10: WS2811C, LED_Driver_KSL:SOP-8_L4.9-W3.9-P1.27-LS6.0-BL, F.Cu at (471.1, 98.8)
- added U11: WS2811C, LED_Driver_KSL:SOP-8_L4.9-W3.9-P1.27-LS6.0-BL, F.Cu at (477.4, 98.8)
- added U12: WS2811C, LED_Driver_KSL:SOP-8_L4.9-W3.9-P1.27-LS6.0-BL, F.Cu at (483.6, 98.8)
- added U13: WS2811C, LED_Driver_KSL:SOP-8_L4.9-W3.9-P1.27-LS6.0-BL, F.Cu at (489.9, 98.8)
- added U14: TPS82130SILR, DC-DC_converter_KSL:USIP-8_L3.0-W2.8-P0.65-TL-EP, F.Cu at (380.7, 85.4)
- added U6: TSSP77038TR, Sensor_KSL:SENSOR-SMD_TSOP75238TR, F.Cu at (457.6, 123.9)
- added U7: TSSP77038TR, Sensor_KSL:SENSOR-SMD_TSOP75238TR, F.Cu at (457.6, 128.5)
- added U8: TSSP77038TR, Sensor_KSL:SENSOR-SMD_TSOP75238TR, F.Cu at (457.6, 133.1)
- added U9: WS2811C, LED_Driver_KSL:SOP-8_L4.9-W3.9-P1.27-LS6.0-BL, F.Cu at (464.8, 98.8)
- C14, C15: value 470uF -> 100nF; footprint Capacitor_THT:C_Radial_D8.0mm_H11.5mm_P3.50mm -> Capacitor_SMD:C_0603_1608Metric_Pad1.08x0.95mm_HandSolder
- C23: value 220uF -> 100nF; footprint Capacitor_THT:C_Radial_D6.3mm_H11.0mm_P2.50mm -> Capacitor_SMD:C_0603_1608Metric_Pad1.08x0.95mm_HandSolder
- C25: value 100nF -> 10uF; footprint Capacitor_SMD:C_0603_1608Metric_Pad1.08x0.95mm_HandSolder -> Capacitor_SMD:C_0805_2012Metric
- C29: value 100nF -> 470pF; footprint Capacitor_SMD:C_0603_1608Metric_Pad1.08x0.95mm_HandSolder -> Capacitor_SMD:C_0603_1608Metric
- D1: value LED yellow -> XL-3210RGBC-YG; footprint LED_SMD:LED_0603_1608Metric -> LED_KSL:LED-ARRAY-SMD_HS-1204-RGB
- D10, D5, D7, D9: value WS2812B -> XL-3210RGBC-YG; footprint LED_SMD:LED_WS2812B_PLCC4_5.0x5.0mm_P3.2mm -> LED_KSL:LED-ARRAY-SMD_HS-1204-RGB
- D2: value 1N4148W -> LED; footprint Diode_SMD:D_SOD-123F -> LED_SMD:LED_0603_1608Metric
- J1: value Conn_01x03 -> USB-TYPE-C-018; footprint Connector_PinHeader_2.54mm:PinHeader_1x03_P2.54mm_Vertical -> Connector_KSL:USB-C_SMD-TYPE-C-31-M-12
- J2: value Conn_01x08 -> GT-BTP30002-0350B-019B; footprint Connector_PinHeader_2.54mm:PinHeader_1x08_P2.54mm_Horizontal -> Connector_KSL:CONN-SMD_GT-BTP30002-0350B-019B; moved to F.Cu
- J3: value Conn_01x02 -> TF_PUSH; footprint Connector_PinHeader_2.54mm:PinHeader_1x02_P2.54mm_Vertical -> Connector_KSL:TF-SMD_TF-PUSH
- J4: value 65100516121 -> GT-BTP30002-0350B-019B; footprint ConnectorsEvo:USB_Mini-B_Wuerth_65100516121_Horizontal -> Connector_KSL:CONN-SMD_GT-BTP30002-0350B-019B
- J5: value Conn_01x05 -> PZ254V-11-04P_C2691448; footprint Connector_PinHeader_2.54mm:PinHeader_1x05_P2.54mm_Vertical -> Connector_KSL:HDR-TH_4P-P2.54-V-M
- R26: footprint Resistor_SMD:R_0603_1608Metric_Pad0.98x0.95mm_HandSolder -> Resistor_SMD:R_0603_1608Metric
- SW1: value SW_DPST_x2 -> SS-12D11G5R; footprint Button_Switch_THT:SW_Slide_SPDT_Straight_CK_OS102011MS2Q -> Switch_KSL:SW-TH_SS-12D11G5R
- SW2: footprint Button_Switch_SMD:SW_Push_1P1T_XKB_TS-1187A -> Button_Switch_SMD:SW_Push_1TS009xxxx-xxxx-xxxx_6x6x5mm
- SW3, SW4: value SW_Push -> SPVN310101; footprint Button_Switch_SMD:SW_Push_1P1T_XKB_TS-1187A -> Switch_KSL:SW-SMD_SPVN310101
- U3: footprint Carte_Mere_PAMI_2025:ESP32-S3-WROOM-1-N16R8 -> MCU_KSL:WIRELM-SMD_ESP32-S3-WROOM-1
- U4, U5: value TMC2226 -> TSSP77038TR; footprint Carte_Mere_PAMI_2025:TMC2226_SHIELD -> Sensor_KSL:SENSOR-SMD_TSOP75238TR
- moved J5 413.4 mm to (515.4, 94.9), turned to 0 degrees
- moved C22 408.9 mm to (481.9, 135.7), turned to 0 degrees
- moved D7 407.1 mm to (472.1, 134.8), turned to 0 degrees
- moved C4 401.0 mm to (493.2, 76.3), turned to 0 degrees
- moved C14 397.3 mm to (467.1, 85.5), turned to 0 degrees
- moved C2 395.3 mm to (493.2, 73.2)
- moved R25 389.7 mm to (480.2, 80.5), turned to 0 degrees
- moved U4 388.2 mm to (457.6, 114.8)
- moved D1 387.9 mm to (472.1, 126.0)
- moved R23 387.9 mm to (480.2, 75.5), turned to 0 degrees
- moved R19 386.4 mm to (475.8, 90.6)
- moved H4 384.2 mm to (465.7, 130.8)
- moved C28 382.6 mm to (471.5, 83.0), turned to 0 degrees
- moved D6 382.5 mm to (493.7, 88.5), turned to 0 degrees
- moved R12 380.1 mm to (475.8, 73.0), turned to 0 degrees
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Connections:
- C10 pad 1: /COLORSIDE -> /BTN_USER1
- C14 pad 1: VBATT_12V -> /BTN_USER2
- C15 pad 1: VBATT_12V -> /uSW4
- C2 pad 1: +5L -> Net-(JP1-C)
- C23 pad 1: +5P -> /uSW5
- C25 pad 1: /PWM_LIDAR -> /VBATT_7V
- C25 pad 2: GND -> GNDPWR
- C29 pad 1: /AU_STATUS -> Net-(U2-SS/TR)
- C29 pad 2: GND -> GNDPWR
- D1 pad 1: GND -> unconnected-(D1-Pad1)
- D1 pad 2: Net-(D1-A) -> unconnected-(D1-Pad2)
- D10 pad 1: +5L -> unconnected-(D10-Pad1)
- D10 pad 2: /WS_5 -> unconnected-(D10-Pad2)
- D10 pad 3: GND -> unconnected-(D10-Pad3)
- D10 pad 4: /WS_4 -> unconnected-(D10-Pad4)
- D2 pad 1: +5P -> Net-(D2-K)
- D2 pad 2: Net-(D2-A) -> +5L
- D5 pad 1: +5L -> unconnected-(D5-Pad1)
- D5 pad 2: /WS_2 -> unconnected-(D5-Pad2)
- D5 pad 3: GND -> unconnected-(D5-Pad3)
- D5 pad 4: /WS_1 -> unconnected-(D5-Pad4)
- D7 pad 1: +5L -> unconnected-(D7-Pad1)
- D7 pad 2: /WS_3 -> unconnected-(D7-Pad2)
- D7 pad 3: GND -> unconnected-(D7-Pad3)
- D7 pad 4: /WS_2 -> unconnected-(D7-Pad4)
- D9 pad 1: +5L -> unconnected-(D9-Pad1)
- D9 pad 2: /WS_4 -> unconnected-(D9-Pad2)
- D9 pad 3: GND -> unconnected-(D9-Pad3)
- D9 pad 4: /WS_3 -> unconnected-(D9-Pad4)
- J1 pad 1: +3.3V -> (no net)
- J1 pad 2: GND -> unconnected-(J1-SH-Pad2)
- J1 pad 3: /TIRETTE -> unconnected-(J1-SH-Pad3)
- J2 pad 1: +5L -> unconnected-(J2-Pad1)
- J2 pad 2: GND -> unconnected-(J2-Pad2)
- J2 pad 3: GND -> unconnected-(J2-Pad3)
- J3 pad 1: Net-(D2-A) -> unconnected-(J3-DAT2-Pad1)
- J3 pad 2: +5P -> unconnected-(J3-CD/DAT3-Pad2)
- J4 pad 1: /5V_USB -> unconnected-(J4-Pad1)
- J4 pad 2: /USB_N -> unconnected-(J4-Pad2)
- J4 pad 3: /USB_P -> unconnected-(J4-Pad3)
- J5 pad 1: /5V_USB -> GND
- J5 pad 2: /USB_N -> +3.3V
- J5 pad 3: /USB_P -> /SCL
- J5 pad 4: GND -> /SDA
- R15 pad 1: /WS_1 -> unconnected-(R15-Pad1)
- R18 pad 1: GND -> /uSW4
- R18 pad 2: /AU_STATUS -> +3.3V
- R20 pad 1: GND -> /uSW5
- R20 pad 2: /PWM_LIDAR -> +3.3V
- R26 pad 1: /AU_STATUS -> Net-(U2-EN)
- R26 pad 2: +5P -> +5VL
- SW1 pad 1: /ALIM_EN_5L -> unconnected-(SW1-Pad1)
- SW1 pad 2: /EN_5L -> unconnected-(SW1-Pad2)
- SW1 pad 3: /EN_5L -> unconnected-(SW1-Pad3)
- SW2 pad 1: /BOOT0 -> /BTN_USER2
- SW3 pad 1: /ESP32_EN -> unconnected-(SW3-Pad1)
- SW3 pad 2: GND -> unconnected-(SW3-Pad2)
- SW4 pad 1: /COLORSIDE -> unconnected-(SW4-Pad1)
- SW4 pad 2: GND -> unconnected-(SW4-Pad2)
- SW7 pad 1: /COLORSIDE -> /BTN_USER1
- U1 pad 3: +5L -> Net-(JP1-C)
- U4 pad 1: GND -> unconnected-(U4-GND-Pad1)
- U4 pad 2: +3.3V -> unconnected-(U4-+VS-Pad2)
- U4 pad 3: Net-(J9-Pin_4) -> unconnected-(U4-OUT-Pad3)
- U4 pad 4: Net-(J9-Pin_3) -> unconnected-(U4-GND-Pad4)
- U5 pad 1: GND -> unconnected-(U5-GND-Pad1)
- U5 pad 2: +3.3V -> unconnected-(U5-+VS-Pad2)
- U5 pad 3: Net-(J10-Pin_4) -> unconnected-(U5-OUT-Pad3)
- U5 pad 4: Net-(J10-Pin_3) -> unconnected-(U5-GND-Pad4)
Routing:
- net GND: track 803.5 -> 0.00 mm, vias 211 -> 0
- net +3.3V: track 346.7 -> 0.00 mm, vias 21 -> 0
- net +5L: track 194.5 -> 0.00 mm, vias 6 -> 0
- net /M_EN: track 158.3 -> 0.00 mm, vias 3 -> 0
- net +5P: track 157.6 -> 0.00 mm, vias 2 -> 0
- net VBATT_12V: track 103.2 -> 0.00 mm
- net /WS_2: track 98.7 -> 0.00 mm, vias 2 -> 0
- net /SERVO1: track 76.0 -> 0.00 mm, vias 2 -> 0
- net /SERVO2: track 73.3 -> 0.00 mm, vias 2 -> 0
- net Net-(Q1-G): track 67.6 -> 0.00 mm, vias 2 -> 0
- net /ALIM_EN_5L: track 67.5 -> 0.00 mm, vias 3 -> 0
- net /EN_5L: track 66.6 -> 0.00 mm, vias 3 -> 0
- net /uSW3: track 65.1 -> 0.00 mm
- net /SDA: track 60.4 -> 0.00 mm, vias 1 -> 0
- net /M1_DIR: track 59.8 -> 0.00 mm, vias 2 -> 0
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- removed copper zone on B.Cu, net GND
- removed copper zone on F.Cu, net GND
Other:
- board size 100 x 77 mm -> 393.2 x 93.1 mm
- board text removed: "+"
- board text removed: "-"
- board text removed: "3L EN TX RX BT GND"
- board text removed: "5-36V"
- board text removed: "5P GND"
- board text removed: "5P GND PWM TXL"
- board text removed: "<= Glory hole"
- board text removed: "Audran"
- board text removed: "BOOT0"
- board text removed: "BTN"
- board text removed: "Bumper AvD"
- board text removed: "Bumper AvG"
- board text removed: "COLOR"
- board text removed: "Carte PAMI 2025"
- board text removed: "Combien d'équipes faut-il pour faire une carte de PAMI pour la coupe IDF?"
- board text removed: "DEBUG"
- board text removed: "Detec. rampe"
- board text removed: "EN_5L Cp2 Cp1 +5P GND GND +5L"
- board text removed: "ERROR"
- board text removed: "GND 5L DI"
- board text removed: "GND 5P S"
- board text removed: "ID"
- board text removed: "LEDs"
- board text removed: "LIDAR LD06"
- board text removed: "M1B M1A M2A M2B"
- board text removed: "MOT Droit"
- board text removed: "MOT Gauche"
- board text removed: "Moteur Fête"
- board text removed: "NC"
- board text removed: "OFF/ON"
- board text removed: "POWER (AU)"
- board text removed: "PWR"
- board text removed: "RESET"
- board text removed: "Servo2 Servo1"
- board text removed: "Servo4 Servo3"
- board text removed: "USB"
- board text removed: "réponse:"
- board text removed: "six: VRAC,Karibous,TDS,Krabi,CHAT,RCVA"

Commit message: Continue PCB placement
Parts:
- removed U14: TPS82130SILR, DC-DC_converter_KSL:USIP-8_L3.0-W2.8-P0.65-TL-EP
- added J10: GT-BTP30002-0350B-019B, Connector_KSL:CONN-SMD_GT-BTP30002-0350B-019B, F.Cu at (20.0, 68.2)
- added J7: GT-BTP30002-0350B-019B, Connector_KSL:CONN-SMD_GT-BTP30002-0350B-019B, F.Cu at (12.7, 58.2)
- added J8: GT-BTP30002-0350B-019B, Connector_KSL:CONN-SMD_GT-BTP30002-0350B-019B, F.Cu at (20.0, 58.2)
- added J9: GT-BTP30002-0350B-019B, Connector_KSL:CONN-SMD_GT-BTP30002-0350B-019B, F.Cu at (12.7, 68.2)
- added U2: TPS82130, DC-DC_converter_KSL:USIP-8_L3.0-W2.8-P0.65-TL-EP, F.Cu at (377.0, 84.1)
- J2, J4: moved to B.Cu
- J5: footprint Connector_KSL:HDR-TH_4P-P2.54-V-M -> Screen_KSL:Waveshare_screen_0.9
- SW1: value SS-12D11G5R -> MSK-22D18G4_051; footprint Switch_KSL:SW-TH_SS-12D11G5R -> Switch_KSL:SW-TH_HX-MSK-22D18G4-051
- moved H6 410.6 mm to (22.8, 132.0)
- moved H7 379.5 mm to (52.8, 53.5)
- moved H5 351.3 mm to (80.3, 104.0)
- moved H9 347.8 mm to (93.8, 132.0)
- moved H8 315.1 mm to (123.8, 53.5)
- moved H10 287.1 mm to (151.3, 104.0)
- moved H12 285.2 mm to (164.8, 132.0)
- moved H13 253.8 mm to (194.8, 53.5)
- moved H11 225.3 mm to (222.3, 104.0)
- moved H16 221.5 mm to (235.8, 132.0)
- moved H15 190.0 mm to (265.8, 53.5)
- moved H17 170.2 mm to (293.3, 104.0)
- moved H14 157.1 mm to (306.8, 132.0)
- moved J5 140.6 mm to (379.9, 132.3)
- moved H19 129.8 mm to (336.8, 53.5)
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Other:
- outline, holes or cut-outs redrawn

Commit message: PCB placement 80%
Parts:
- removed H1, H2, H3, H4: MountingHole_Pad, MountingHole:MountingHole_3.2mm_M3_Pad
- removed SW2, SW5, SW6, SW7: SW_Push, Button_Switch_SMD:SW_Push_1TS009xxxx-xxxx-xxxx_6x6x5mm
- added REF**: MountingHole_3.2mm_M3, MountingHole:MountingHole_3.2mm_M3, F.Cu at (406.5, 99.5)
- added REF**: MountingHole_3.2mm_M3, MountingHole:MountingHole_3.2mm_M3, F.Cu at (397.5, 124.0)
- moved D1 449.5 mm to (28.0, 56.2), turned to -135 degrees
- moved SW3 438.5 mm to (34.8, 134.0), turned to -45 degrees
- moved U6 434.9 mm to (23.9, 92.1), turned to -135 degrees
- moved D4 401.0 mm to (77.7, 56.2), turned to 135 degrees
- moved D5 380.6 mm to (99.0, 56.2), turned to -135 degrees
- moved U9 378.5 mm to (88.0, 63.4), turned to -90 degrees
- moved SW4 373.3 mm to (105.7, 134.0), turned to -45 degrees
- moved U5 363.7 mm to (94.9, 92.1), turned to -135 degrees
- moved D7 332.8 mm to (148.6, 56.2), turned to 135 degrees
- moved U10 313.8 mm to (159.3, 63.5), turned to -90 degrees
- moved D9 312.9 mm to (169.9, 56.2), turned to -135 degrees
- moved SW8 308.2 mm to (176.7, 134.0), turned to -45 degrees
- moved U4 292.6 mm to (165.9, 92.1), turned to -135 degrees
- moved D10 266.2 mm to (219.6, 56.2), turned to 135 degrees
- moved U11 249.6 mm to (230.3, 63.4), turned to -90 degrees
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Other:
- board size 393.2 x 93.1 mm -> 409.4 x 93 mm
- board text added: "GND"
- board text added: "VBAT+"

Commit message: Schematics done 90% + PCB placement +10%
Parts:
- removed REF** (x2): MountingHole_3.2mm_M3, MountingHole:MountingHole_3.2mm_M3
- added D15: 1N4148W, Diode_SMD:D_SOD-123F, F.Cu at (446.1, 99.5)
- added H1: SMTSO3040CTJ, Fastener_KSL:SMD-1_BD5.5-D4.0, F.Cu at (406.0, 97.6)
- added H2: SMTSO3040CTJ, Fastener_KSL:SMD-1_BD5.5-D4.0, F.Cu at (395.0, 123.1)
- added H3: SMTSO3040CTJ, Fastener_KSL:SMD-1_BD5.5-D4.0, F.Cu at (439.5, 92.8)
- added H4: SMTSO3040CTJ, Fastener_KSL:SMD-1_BD5.5-D4.0, F.Cu at (437.9, 103.1)
- added R1: 5.1k, Resistor_SMD:R_0603_1608Metric, F.Cu at (451.9, 75.0)
- added R2: 4.7k, Resistor_SMD:R_0603_1608Metric, F.Cu at (451.9, 77.5)
- added R3: 5.1k, Resistor_SMD:R_0603_1608Metric, F.Cu at (451.9, 80.0)
- added R4: 1k, Resistor_SMD:R_0603_1608Metric, F.Cu at (451.9, 82.5)
- added R5: 68, Resistor_SMD:R_0603_1608Metric, F.Cu at (451.9, 85.0)
- added R6: 68, Resistor_SMD:R_0603_1608Metric, F.Cu at (451.9, 87.5)
- added SW15: SPVN310101, Switch_KSL:SW-SMD_SPVN310101, F.Cu at (29.3, 109.0)
- added SW2: TS-1088-AR02016, Switch_KSL:SW-SMD_L3.9-W3.0-P4.45, F.Cu at (391.5, 113.4)
- added SW5: TS-1088-AR02016, Switch_KSL:SW-SMD_L3.9-W3.0-P4.45, F.Cu at (383.5, 113.4)
- added SW6: TS-1088-AR02016, Switch_KSL:SW-SMD_L3.9-W3.0-P4.45, F.Cu at (383.5, 89.1)
- added SW7: TS-1088-AR02016, Switch_KSL:SW-SMD_L3.9-W3.0-P4.45, F.Cu at (375.5, 113.3)
- SW11, SW12, SW13, SW14: value TS-1088-AR02016 -> SPVN310101; footprint Switch_KSL:SW-SMD_L3.9-W3.0-P4.45 -> Switch_KSL:SW-SMD_SPVN310101
- moved SW14 277.8 mm to (100.3, 109.0), turned to -90 degrees
- moved SW13 206.6 mm to (171.3, 109.0), turned to -90 degrees
- moved SW12 140.4 mm to (242.3, 109.0)
- moved SW11 97.9 mm to (313.3, 109.0), turned to -90 degrees
Connections:
- C25 pad 2: GNDPWR -> GND
- C29 pad 2: GNDPWR -> GND
- C30 pad 2: GNDPWR -> GND
- C8 pad 1: /5V_USB -> /VBUS
- H10 pad 1: unconnected-(H10-Pad1) -> GND
- H11 pad 1: unconnected-(H11-Pad1) -> GND
- H12 pad 1: unconnected-(H12-Pad1) -> GND
- H13 pad 1: unconnected-(H13-Pad1) -> GND
- H14 pad 1: unconnected-(H14-Pad1) -> GND
- H15 pad 1: unconnected-(H15-Pad1) -> GND
- H5 pad 1: unconnected-(H5-Pad1) -> GND
- H6 pad 1: unconnected-(H6-Pad1) -> GND
- H7 pad 1: unconnected-(H7-Pad1) -> GND
- H8 pad 1: unconnected-(H8-Pad1) -> GND
- H9 pad 1: unconnected-(H9-Pad1) -> GND
- J1 pad 0: unconnected-(J1-SH-Pad0) -> GND
- J1 pad 2: unconnected-(J1-SH-Pad2) -> GND
- J1 pad 3: unconnected-(J1-SH-Pad3) -> GND
- J1 pad A1: unconnected-(J1-GND-PadA1) -> GND
- J1 pad A12: unconnected-(J1-GND-PadA12) -> GND
- J1 pad A4: unconnected-(J1-VBUS-PadA4) -> /VBUS
- J1 pad A5: unconnected-(J1-CC1-PadA5) -> /CC1
- J1 pad A6: unconnected-(J1-DP1-PadA6) -> /USB_P
- J1 pad A7: unconnected-(J1-DN1-PadA7) -> /USB_N
- J1 pad A9: unconnected-(J1-VBUS-PadA9) -> /VBUS
- J1 pad B1: unconnected-(J1-GND-PadB1) -> GND
- J1 pad B12: unconnected-(J1-GND-PadB12) -> GND
- J1 pad B4: unconnected-(J1-VBUS-PadB4) -> /VBUS
- J1 pad B5: unconnected-(J1-CC2-PadB5) -> /CC2
- J1 pad B6: unconnected-(J1-DP2-PadB6) -> /USB_P
- J1 pad B7: unconnected-(J1-DN2-PadB7) -> /USB_N
- J1 pad B9: unconnected-(J1-VBUS-PadB9) -> /VBUS
- J2 pad 2: unconnected-(J2-Pad2) -> GND
- J4 pad 1: unconnected-(J4-Pad1) -> /VBATT_7V
- R27 pad 1: GNDPWR -> GND
- R27 pad 2: Net-(U2-EN) -> /EN_5L
- R28 pad 1: +5VP -> +5L
- R31 pad 1: GNDPWR -> GND
- SW1 pad 1: unconnected-(SW1-Pad1) -> /VBATT_7V
- SW1 pad 2: unconnected-(SW1-Pad2) -> /VBATT_7V
- SW1 pad 3: unconnected-(SW1-Pad3) -> /SWITCHED_7V
- SW1 pad 4: unconnected-(SW1-Pad4) -> /VBATT_7V
- SW1 pad 5: unconnected-(SW1-Pad5) -> /VBATT_7V
- SW1 pad 6: unconnected-(SW1-Pad6) -> /SWITCHED_7V
- SW10 pad 1: unconnected-(SW10-Pad1) -> /uSW3
- SW10 pad 2: unconnected-(SW10-Pad2) -> GND
- SW10 pad 3: unconnected-(SW10-Pad3) -> GND
- SW10 pad 4: unconnected-(SW10-Pad4) -> /uSW3
- SW11 pad 1: unconnected-(SW11-Pad1) -> /uSW3
- SW11 pad 2: unconnected-(SW11-Pad2) -> GND
- SW12 pad 1: unconnected-(SW12-Pad1) -> /uSW4
- SW12 pad 2: unconnected-(SW12-Pad2) -> GND
- SW13 pad 1: unconnected-(SW13-Pad1) -> /uSW4
- SW13 pad 2: unconnected-(SW13-Pad2) -> GND
- SW14 pad 1: unconnected-(SW14-Pad1) -> /uSW5
- SW14 pad 2: unconnected-(SW14-Pad2) -> GND
- SW3 pad 1: unconnected-(SW3-Pad1) -> /uSW1
- SW3 pad 2: unconnected-(SW3-Pad2) -> GND
- SW3 pad 3: unconnected-(SW3-Pad3) -> GND
- SW3 pad 4: unconnected-(SW3-Pad4) -> /uSW1
- SW4 pad 1: unconnected-(SW4-Pad1) -> /uSW1
- SW4 pad 2: unconnected-(SW4-Pad2) -> GND
- SW4 pad 3: unconnected-(SW4-Pad3) -> GND
- SW4 pad 4: unconnected-(SW4-Pad4) -> /uSW1
- SW8 pad 1: unconnected-(SW8-Pad1) -> /uSW2
- SW8 pad 2: unconnected-(SW8-Pad2) -> GND
- SW8 pad 3: unconnected-(SW8-Pad3) -> GND
- SW8 pad 4: unconnected-(SW8-Pad4) -> /uSW2
- SW9 pad 1: unconnected-(SW9-Pad1) -> /uSW2
- SW9 pad 2: unconnected-(SW9-Pad2) -> GND
- SW9 pad 3: unconnected-(SW9-Pad3) -> GND
- SW9 pad 4: unconnected-(SW9-Pad4) -> /uSW2
- U2 pad 1: Net-(U2-EN) -> /EN_5L
- U2 pad 3: GNDPWR -> GND
- U2 pad 9: GNDPWR -> GND
Other:
- outline, holes or cut-outs redrawn
- board text added: "B0"
- board text added: "↵"

Commit message: Placement done
Parts:
- removed BZ1: Buzzer, Buzzer_Beeper:Buzzer_TDK_PS1240P02BT_D12.2mm_H6.5mm
- removed D6: 1N4148W, Diode_SMD:D_SOD-123F
- removed H2, H4: SMTSO3040CTJ, Fastener_KSL:SMD-1_BD5.5-D4.0
- removed Q2: G2302, Package_TO_SOT_SMD:SOT-23
- removed R14: 10k, Resistor_SMD:R_0603_1608Metric_Pad0.98x0.95mm_HandSolder
- added C1: 22uF, Capacitor_SMD:C_0805_2012Metric, F.Cu at (17.2, 85.8)
- added C16: 22uF, Capacitor_SMD:C_0805_2012Metric, F.Cu at (301.3, 84.7)
- added C19: 100n, Capacitor_SMD:C_0603_1608Metric_Pad1.08x0.95mm_HandSolder, F.Cu at (235.0, 61.6)
- added C20: 100n, Capacitor_SMD:C_0603_1608Metric_Pad1.08x0.95mm_HandSolder, F.Cu at (306.1, 61.9)
- added C21: 100n, Capacitor_SMD:C_0603_1608Metric_Pad1.08x0.95mm_HandSolder, F.Cu at (376.5, 61.5)
- added C24: 100n, Capacitor_SMD:C_0603_1608Metric_Pad1.08x0.95mm_HandSolder, F.Cu at (92.8, 61.9)
- added C3: 22uF, Capacitor_SMD:C_0805_2012Metric, F.Cu at (88.5, 85.8)
- added C31: 22uF, Capacitor_SMD:C_0805_2012Metric, F.Cu at (167.0, 50.9)
- added C31: 22uF, Capacitor_SMD:C_0805_2012Metric, F.Cu at (161.7, 121.6)
- added C5: 22uF, Capacitor_SMD:C_0805_2012Metric, F.Cu at (159.5, 85.8)
- added C6: 22uF, Capacitor_SMD:C_0805_2012Metric, F.Cu at (230.5, 85.8)
- added JP2: SolderJumper_3_Bridged12, Jumper:SolderJumper-3_P1.3mm_Bridged12_RoundedPad1.0x1.5mm, F.Cu at (384.0, 69.0)
- added Q1: 2N7002, Package_TO_SOT_SMD:SOT-23_Handsoldering, F.Cu at (382.0, 64.0)
- added R21: 33, Resistor_SMD:R_0603_1608Metric, F.Cu at (80.2, 54.1)
- added R22: 33, Resistor_SMD:R_0603_1608Metric, F.Cu at (79.4, 51.8)
- added R33: 33, Resistor_SMD:R_0603_1608Metric, F.Cu at (152.0, 56.0)
- added R34: 33, Resistor_SMD:R_0603_1608Metric, F.Cu at (221.8, 52.3)
- added R35: 33, Resistor_SMD:R_0603_1608Metric, F.Cu at (222.4, 54.4)
- added R36: 33, Resistor_SMD:R_0603_1608Metric, F.Cu at (223.2, 56.3)
- added R37: 33, Resistor_SMD:R_0603_1608Metric, F.Cu at (292.5, 51.8)
- added R38: 33, Resistor_SMD:R_0603_1608Metric, F.Cu at (293.1, 53.6)
- added R39: 33, Resistor_SMD:R_0603_1608Metric, F.Cu at (293.8, 55.3)
- added R40: 33, Resistor_SMD:R_0603_1608Metric, F.Cu at (363.8, 51.8)
- added R41: 33, Resistor_SMD:R_0603_1608Metric, F.Cu at (364.4, 53.8)
- added R42: 33, Resistor_SMD:R_0603_1608Metric, F.Cu at (365.2, 55.8)
- added R43: 4.7k, Resistor_SMD:R_0603_1608Metric, F.Cu at (380.5, 126.0)
- added R7: 33, Resistor_SMD:R_0603_1608Metric, F.Cu at (81.2, 56.2)
- added R8: 150, Resistor_SMD:R_0603_1608Metric, F.Cu at (93.5, 59.2)
- added REF**: MountingHole_3.2mm_M3, MountingHole:MountingHole_3.2mm_M3, F.Cu at (395.0, 123.1)
- added REF**: MountingHole_3.2mm_M3, MountingHole:MountingHole_3.2mm_M3, F.Cu at (406.1, 97.6)
- added U14: TSSP77038TT, Sensor_KSL:Top-view-TSSP770_SMD_TSOP75238TR, F.Cu at (166.5, 120.7)
- added U14: TSSP77038TT, Sensor_KSL:Top-view-TSSP770_SMD_TSOP75238TR, F.Cu at (172.0, 51.7)
- C18: value 100nF -> 100n
- R10, R11: value 10k -> 4.7k; footprint Resistor_SMD:R_0603_1608Metric_Pad0.98x0.95mm_HandSolder -> Resistor_SMD:R_0603_1608Metric
- R12: footprint Resistor_SMD:R_0603_1608Metric_Pad0.98x0.95mm_HandSolder -> Resistor_SMD:R_0603_1608Metric
- R15: value 68 -> 150; footprint Resistor_SMD:R_0603_1608Metric_Pad0.98x0.95mm_HandSolder -> Resistor_SMD:R_0603_1608Metric
- R16: value 10k -> 150; footprint Resistor_SMD:R_0603_1608Metric_Pad0.98x0.95mm_HandSolder -> Resistor_SMD:R_0603_1608Metric
- R17, R9: value 1k -> 150; footprint Resistor_SMD:R_0603_1608Metric_Pad0.98x0.95mm_HandSolder -> Resistor_SMD:R_0603_1608Metric
- R26: value 10k -> 33
- R32: value 4.7k -> 33
- R5, R6: value 68 -> 33
- moved R32 335.5 mm to (150.9, 53.8), turned to 45 degrees
- moved R26 335.2 mm to (150.0, 51.4), turned to 45 degrees
- moved R9 307.8 mm to (164.8, 59.2)
- moved C18 307.7 mm to (164.0, 61.9), turned to 90 degrees
- moved R15 241.0 mm to (235.8, 59.0)
- moved R16 170.5 mm to (307.0, 59.2)
- moved C11 126.6 mm to (380.0, 52.7), turned to 90 degrees
- moved C22 113.9 mm to (374.5, 97.8), turned to -90 degrees
- moved C2 112.9 mm to (381.5, 56.2), turned to 180 degrees
- moved R17 104.8 mm to (374.5, 58.8), turned to 90 degrees
- moved D3 102.8 mm to (372.2, 52.7)
- moved R10 101.8 mm to (377.0, 126.0), turned to 180 degrees
- moved R19 101.4 mm to (376.0, 72.8)
- moved C4 100.8 mm to (394.2, 56.8)
- moved C25 100.3 mm to (394.0, 97.5)
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Connections:
- net /COLORSIDE renamed /CARD_DETECT
- C18 pad 1: +5P -> GND
- C18 pad 2: GND -> Net-(U10-VDD)
- C22 pad 1: +5P -> +5L
- D1 pad 1: unconnected-(D1-Pad1) -> Net-(D1-B)
- D1 pad 2: unconnected-(D1-Pad2) -> Net-(D1-G)
- D1 pad 3: unconnected-(D1-Pad3) -> +5L
- D1 pad 4: unconnected-(D1-Pad4) -> Net-(D1-R)
- D10 pad 1: unconnected-(D10-Pad1) -> Net-(D10-B)
- D10 pad 2: unconnected-(D10-Pad2) -> Net-(D10-G)
- D10 pad 3: unconnected-(D10-Pad3) -> +5L
- D10 pad 4: unconnected-(D10-Pad4) -> Net-(D10-R)
- D11 pad 1: unconnected-(D11-Pad1) -> Net-(D11-B)
- D11 pad 2: unconnected-(D11-Pad2) -> Net-(D11-G)
- D11 pad 3: unconnected-(D11-Pad3) -> +5L
- D11 pad 4: unconnected-(D11-Pad4) -> Net-(D11-R)
- D12 pad 1: unconnected-(D12-Pad1) -> Net-(D11-B)
- D12 pad 2: unconnected-(D12-Pad2) -> Net-(D11-G)
- D12 pad 3: unconnected-(D12-Pad3) -> +5L
- D12 pad 4: unconnected-(D12-Pad4) -> Net-(D11-R)
- D13 pad 1: unconnected-(D13-Pad1) -> Net-(D13-B)
- D13 pad 2: unconnected-(D13-Pad2) -> Net-(D13-G)
- D13 pad 3: unconnected-(D13-Pad3) -> +5L
- D13 pad 4: unconnected-(D13-Pad4) -> Net-(D13-R)
- D14 pad 1: unconnected-(D14-Pad1) -> Net-(D13-B)
- D14 pad 2: unconnected-(D14-Pad2) -> Net-(D13-G)
- D14 pad 3: unconnected-(D14-Pad3) -> +5L
- D14 pad 4: unconnected-(D14-Pad4) -> Net-(D13-R)
- D4 pad 1: unconnected-(D4-Pad1) -> Net-(D1-B)
- D4 pad 2: unconnected-(D4-Pad2) -> Net-(D1-G)
- D4 pad 3: unconnected-(D4-Pad3) -> +5L
- D4 pad 4: unconnected-(D4-Pad4) -> Net-(D1-R)
- D5 pad 1: unconnected-(D5-Pad1) -> Net-(D5-B)
- D5 pad 2: unconnected-(D5-Pad2) -> Net-(D5-G)
- D5 pad 3: unconnected-(D5-Pad3) -> +5L
- D5 pad 4: unconnected-(D5-Pad4) -> Net-(D5-R)
- D7 pad 1: unconnected-(D7-Pad1) -> Net-(D5-B)
- D7 pad 2: unconnected-(D7-Pad2) -> Net-(D5-G)
- D7 pad 3: unconnected-(D7-Pad3) -> +5L
- D7 pad 4: unconnected-(D7-Pad4) -> Net-(D5-R)
- D9 pad 1: unconnected-(D9-Pad1) -> Net-(D10-B)
- D9 pad 2: unconnected-(D9-Pad2) -> Net-(D10-G)
- D9 pad 3: unconnected-(D9-Pad3) -> +5L
- D9 pad 4: unconnected-(D9-Pad4) -> Net-(D10-R)
- J11 pad 2: +5P -> +5L
- J3 pad 10: unconnected-(J3-Pad10) -> GND
- J3 pad 11: unconnected-(J3-Pad11) -> GND
- J3 pad 12: unconnected-(J3-Pad12) -> GND
- J3 pad 13: unconnected-(J3-Pad13) -> GND
- J3 pad 2: unconnected-(J3-CD/DAT3-Pad2) -> /CS
- J3 pad 3: unconnected-(J3-CMD-Pad3) -> /MOSI
- J3 pad 4: unconnected-(J3-VDD-Pad4) -> +3.3V
- J3 pad 5: unconnected-(J3-CLX-Pad5) -> /SCK
- J3 pad 6: unconnected-(J3-VSS-Pad6) -> GND
- J3 pad 7: unconnected-(J3-DAT0-Pad7) -> /MISO
- R10 pad 1: /SCL -> /SDA
- R11 pad 1: /SCL -> Net-(JP2-A)
- R12 pad 1: /SDA -> /RGBLED
- R12 pad 2: +3.3V -> +5L
- R15 pad 1: unconnected-(R15-Pad1) -> Net-(U11-VDD)
- R15 pad 2: /RGBLED -> +5L
- R16 pad 1: GND -> Net-(U12-VDD)
- R16 pad 2: /BUZZER -> +5L
- R17 pad 1: Net-(BZ1--) -> Net-(U13-VDD)
- R17 pad 2: +5P -> +5L
- R26 pad 1: Net-(U2-EN) -> Net-(D5-B)
- R26 pad 2: +5VL -> Net-(U10-OUTB)
- R32 pad 1: Net-(D2-K) -> Net-(D5-G)
- R32 pad 2: GNDPWR -> Net-(U10-OUTG)
- R5 pad 1: unconnected-(R5-Pad1) -> Net-(U13-DIN)
- R9 pad 1: GND -> Net-(U10-VDD)
- R9 pad 2: Net-(D3-K) -> +5L
- SW10 pad 1: /uSW3 -> /uSW5
- SW10 pad 4: /uSW3 -> Net-(SW10-Pad4)
- SW11 pad 1: /uSW3 -> Net-(SW10-Pad4)
- SW11 pad 4: /uSW3 -> Net-(SW10-Pad4)
- SW13 pad 1: /uSW4 -> /uSW3
- SW13 pad 4: /uSW4 -> /uSW3
- SW14 pad 1: /uSW5 -> /uSW2
- SW14 pad 4: /uSW5 -> /uSW2
- SW15 pad 1: /uSW5 -> /uSW1
- SW15 pad 4: /uSW5 -> /uSW1
- SW4 pad 1: /uSW1 -> /uSW2
- SW4 pad 4: /uSW1 -> /uSW2
- SW8 pad 1: /uSW2 -> /uSW3
- SW8 pad 4: /uSW2 -> /uSW3
- SW9 pad 1: /uSW2 -> /uSW4
- SW9 pad 4: /uSW2 -> /uSW4
- U10 pad 1: unconnected-(U10-OUTR-Pad1) -> Net-(U10-OUTR)
- U10 pad 2: unconnected-(U10-OUTG-Pad2) -> Net-(U10-OUTG)
- U10 pad 3: unconnected-(U10-OUTB-Pad3) -> Net-(U10-OUTB)
- U10 pad 4: unconnected-(U10-GND-Pad4) -> GND
- U10 pad 5: unconnected-(U10-DO-Pad5) -> Net-(U10-DO)
- U10 pad 6: unconnected-(U10-DIN-Pad6) -> Net-(U10-DIN)
- U10 pad 8: unconnected-(U10-VDD-Pad8) -> Net-(U10-VDD)
- U11 pad 1: unconnected-(U11-OUTR-Pad1) -> Net-(U11-OUTR)
- U11 pad 2: unconnected-(U11-OUTG-Pad2) -> Net-(U11-OUTG)
- U11 pad 3: unconnected-(U11-OUTB-Pad3) -> Net-(U11-OUTB)
- U11 pad 4: unconnected-(U11-GND-Pad4) -> GND
- U11 pad 5: unconnected-(U11-DO-Pad5) -> Net-(U10-DIN)
- U11 pad 6: unconnected-(U11-DIN-Pad6) -> Net-(U11-DIN)
- U11 pad 8: unconnected-(U11-VDD-Pad8) -> Net-(U11-VDD)
- U12 pad 1: unconnected-(U12-OUTR-Pad1) -> Net-(U12-OUTR)
- U12 pad 2: unconnected-(U12-OUTG-Pad2) -> Net-(U12-OUTG)
- U12 pad 3: unconnected-(U12-OUTB-Pad3) -> Net-(U12-OUTB)
- U12 pad 4: unconnected-(U12-GND-Pad4) -> GND
- U12 pad 5: unconnected-(U12-DO-Pad5) -> Net-(U11-DIN)
- U12 pad 6: unconnected-(U12-DIN-Pad6) -> Net-(U12-DIN)
- U12 pad 8: unconnected-(U12-VDD-Pad8) -> Net-(U12-VDD)
- U13 pad 1: unconnected-(U13-OUTR-Pad1) -> Net-(U13-OUTR)
- U13 pad 2: unconnected-(U13-OUTG-Pad2) -> Net-(U13-OUTG)
- U13 pad 3: unconnected-(U13-OUTB-Pad3) -> Net-(U13-OUTB)
- U13 pad 4: unconnected-(U13-GND-Pad4) -> GND
- U13 pad 5: unconnected-(U13-DO-Pad5) -> Net-(U12-DIN)
- U13 pad 6: unconnected-(U13-DIN-Pad6) -> Net-(U13-DIN)
- U13 pad 8: unconnected-(U13-VDD-Pad8) -> Net-(U13-VDD)
- U3 pad 11: /SERVO2 -> /BTN_USER2
- U3 pad 12: /M_EN -> /CS
- U3 pad 17: /TIRETTE -> /RGBLED_3V3
- U3 pad 18: /LED_RED -> /BTN_USER1
- U3 pad 21: /uSW3 -> /uSW5
- U3 pad 22: /BUZZER -> /uSW4
- U3 pad 23: /CaptTOR_2 -> /uSW3
- U3 pad 24: /TX_LIDAR -> /uSW2
- U3 pad 25: /M1_STEP -> /uSW1
- U3 pad 31: /M2_STEP -> /IRSENS_1
- U3 pad 32: /M2_DIR -> /IRSENS_2
- U3 pad 33: /SERVO3 -> /IRSENS_3
- U3 pad 34: /CaptTOR_1 -> /IRSENS_4
- U3 pad 35: /SERVO4 -> /IRSENS_5
- U3 pad 38: /M2_DIAG/uSW2 -> /IRSENS_F
- U3 pad 39: /AU_STATUS -> /LED_RED
- U3 pad 5: /RGBLED -> /SCK
- U3 pad 6: /ID2 -> /MOSI
- U3 pad 7: /ID1 -> /MISO
- U3 pad 8: /M1_DIAG/uSW1 -> /ID2
- U3 pad 9: /M1_DIR -> /ID1
- U4 pad 1: unconnected-(U4-GND-Pad1) -> GND
- U4 pad 2: unconnected-(U4-+VS-Pad2) -> +3.3V
- U4 pad 3: unconnected-(U4-OUT-Pad3) -> /IRSENS_3
- U4 pad 4: unconnected-(U4-GND-Pad4) -> GND
- U5 pad 1: unconnected-(U5-GND-Pad1) -> GND
- U5 pad 2: unconnected-(U5-+VS-Pad2) -> +3.3V
- U5 pad 3: unconnected-(U5-OUT-Pad3) -> /IRSENS_2
- U5 pad 4: unconnected-(U5-GND-Pad4) -> GND
- U6 pad 1: unconnected-(U6-GND-Pad1) -> GND
- U6 pad 2: unconnected-(U6-+VS-Pad2) -> +3.3V
- U6 pad 3: unconnected-(U6-OUT-Pad3) -> /IRSENS_1
- U6 pad 4: unconnected-(U6-GND-Pad4) -> GND
- U7 pad 1: unconnected-(U7-GND-Pad1) -> GND
- U7 pad 2: unconnected-(U7-+VS-Pad2) -> +3.3V
- U7 pad 3: unconnected-(U7-OUT-Pad3) -> /IRSENS_4
- U7 pad 4: unconnected-(U7-GND-Pad4) -> GND
- U8 pad 1: unconnected-(U8-GND-Pad1) -> GND
- U8 pad 2: unconnected-(U8-+VS-Pad2) -> +3.3V
- U8 pad 3: unconnected-(U8-OUT-Pad3) -> /IRSENS_5
- U8 pad 4: unconnected-(U8-GND-Pad4) -> GND
- U9 pad 1: unconnected-(U9-OUTR-Pad1) -> Net-(U9-OUTR)
- U9 pad 2: unconnected-(U9-OUTG-Pad2) -> Net-(U9-OUTG)
- U9 pad 3: unconnected-(U9-OUTB-Pad3) -> Net-(U9-OUTB)
- U9 pad 4: unconnected-(U9-GND-Pad4) -> GND
- U9 pad 6: unconnected-(U9-DIN-Pad6) -> Net-(U10-DO)
- U9 pad 8: unconnected-(U9-VDD-Pad8) -> Net-(U9-VDD)
Routing:
- net +3.3V: track 0.00 -> 22.5 mm
- net /RGBLED: track 0.00 -> 7.75 mm
- net Net-(JP2-A): track 0.00 -> 2.60 mm
Other:
- board text added: "3V3 ON"
- board text added: "5V ON"

Commit message: Routing 80%
Parts:
- added J12: LED strip, Connector_PinHeader_2.54mm:PinHeader_1x03_P2.54mm_Vertical, F.Cu at (57.0, 81.5)
- moved R10 79.1 mm to (451.2, 153.2), turned to 90 degrees
- moved R43 77.0 mm to (451.2, 156.5), turned to 90 degrees
- moved U14 44.1 mm to (211.2, 71.7)
- moved C31 43.7 mm to (206.2, 70.2)
- moved J6 42.9 mm to (438.4, 109.0)
- moved R15 42.7 mm to (272.2, 81.2)
- moved U9 42.5 mm to (124.5, 85.2)
- moved C19 42.5 mm to (271.2, 83.8)
- moved U11 42.4 mm to (266.5, 85.5)
- moved U10 42.4 mm to (195.5, 85.5)
- moved U12 42.3 mm to (337.5, 85.2)
- moved C20 42.3 mm to (342.2, 83.9)
- moved R16 42.2 mm to (343.0, 81.2)
- moved C24 42.2 mm to (129.2, 83.1)
- moved R8 42.2 mm to (129.9, 80.5)
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Connections:
- R10 pad 1: /SDA -> /SCL
- R43 pad 1: /SCL -> /SDA
- SW10 pad 4: Net-(SW10-Pad4) -> /uSW5
- SW11 pad 1: Net-(SW10-Pad4) -> /uSW5
- SW11 pad 4: Net-(SW10-Pad4) -> /uSW5
- U3 pad 19: /SDA -> /SCL
- U3 pad 20: /SCL -> /SDA
- U3 pad 5: /SCK -> /MISO
- U3 pad 6: /MOSI -> /SCK
- U3 pad 7: /MISO -> /MOSI
- U9 pad 5: unconnected-(U9-DO-Pad5) -> Net-(J12-Pin_2)
Routing:
- net +3.3V: track 22.5 -> 525.3 mm, vias 0 -> 8
- net /uSW1: track 0.00 -> 416.3 mm, vias 0 -> 2
- net /IRSENS_1: track 0.00 -> 414.2 mm
- net /uSW2: track 0.00 -> 346.2 mm, vias 0 -> 2
- net /IRSENS_2: track 0.00 -> 341.5 mm
- net /uSW3: track 0.00 -> 277.9 mm, vias 0 -> 2
- net /IRSENS_3: track 0.00 -> 268.7 mm
- net +5L: track 0.00 -> 265.4 mm
- net /uSW4: track 0.00 -> 208.6 mm, vias 0 -> 2
- net /IRSENS_4: track 0.00 -> 197.5 mm
- net GND: track 0.00 -> 194.8 mm
- net /uSW5: track 0.00 -> 141.0 mm, vias 0 -> 2
- net /IRSENS_5: track 0.00 -> 119.2 mm
- net /SDA: track 0.00 -> 83.1 mm, vias 0 -> 1
- net /SCL: track 0.00 -> 81.1 mm, vias 0 -> 1
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
Commit message: 90% routing
Parts:
- moved D8 39.8 mm to (447.0, 104.2), turned to 180 degrees
- moved R19 34.6 mm to (445.4, 102.5), turned to 180 degrees
- moved C31 0.75 mm to (205.5, 70.2), turned to 180 degrees
Routing:
- net +5L: track 265.4 -> 795.0 mm, vias 0 -> 10
- net /IRSENS_F: track 0.00 -> 372.5 mm, vias 0 -> 2
- net GND: track 194.8 -> 371.0 mm, vias 0 -> 1
- net +3.3V: track 525.3 -> 690.6 mm, vias 8 -> 14
- net Net-(D11-B): track 0.00 -> 60.5 mm
- net Net-(D11-G): track 0.00 -> 57.7 mm
- net /BTN_USER1: track 0.00 -> 56.2 mm, vias 0 -> 2
- net Net-(D11-R): track 0.00 -> 55.7 mm
- net /SERVO1: track 0.00 -> 40.5 mm, vias 0 -> 1
- net /BOOT0: track 12.7 -> 41.9 mm
- net Net-(U10-VDD): track 0.00 -> 5.21 mm
- net Net-(D2-K): track 0.00 -> 2.25 mm
- net Net-(D8-A): track 0.00 -> 1.78 mm
- net /LED_RED: track 0.00 -> 1.75 mm
- net /MISO: track 62.7 -> 64.2 mm
