File: Satisfactron_2025.kicad_pcb (KiCad board)
At the start: 2 copper layers, 409.4 x 93 mm, 153 parts, among them J1 USB-TYPE-C-018, J10 GT-BTP30002-0350B-019B, J11 Conn_01x03, J12 LED strip, J2 GT-BTP30002-0350B-019B, J3 TF_PUSH, J4 GT-BTP30002-0350B-019B, J5 PZ254V-11-04P_C2691448, J6 Conn_01x06, J7 GT-BTP30002-0350B-019B, J8 GT-BTP30002-0350B-019B, J9 GT-BTP30002-0350B-019B, Q1 2N7002, SW1 MSK-22D18G4_051, SW10 SPVN310101, SW11 SPVN310101, SW12 SPVN310101, SW13 SPVN310101, SW14 SPVN310101, SW15 SPVN310101, SW2 TS-1088-AR02016, SW3 SPVN310101, SW4 SPVN310101, SW5 TS-1088-AR02016, SW6 TS-1088-AR02016, SW7 TS-1088-AR02016, SW8 SPVN310101, SW9 SPVN310101, U1 AMS1117-3.3, U10 WS2811C, U11 WS2811C, U12 WS2811C, U13 WS2811C, U14 TSSP77038TT, U2 TPS82130, U3 ESP32-S3-WROOM-1-N16R8, U4 TSSP77038TR, U5 TSSP77038TR, U6 TSSP77038TR, U7 TSSP77038TR, U8 TSSP77038TR, U9 WS2811C

Commit message: Routing done, no zones
Parts:
- moved JP6 9.58 mm to (434.7, 79.8), turned to -90 degrees
- moved JP7 9.58 mm to (438.2, 79.8), turned to -90 degrees
- moved R19 0.41 mm to (445.0, 102.5)
- moved R6 0.25 mm to (425.2, 123.0)
Connections:
- J1 pad 1: (no net) -> GND
Routing:
- net GND: track 371.0 -> 1977.7 mm, vias 1 -> 41
- net /VBUS: track 0.00 -> 16.6 mm
- net +3.3V: track 690.6 -> 702.5 mm
- net +5L: track 795.0 -> 789.1 mm, vias 10 -> 11
- net /USB_P: track 50.2 -> 55.6 mm
- net /USB_N: track 48.1 -> 52.2 mm, vias 2 -> 4
- net /uSW3: track 277.9 -> 281.9 mm, vias 2 -> 4
- net /uSW4: track 208.6 -> 212.3 mm, vias 2 -> 4
- net /ID2: track 0.00 -> 3.42 mm
- net /uSW5: track 141.0 -> 144.3 mm, vias 2 -> 4
- net /ID1: track 0.00 -> 3.22 mm
- net Net-(D3-K): track 0.00 -> 2.74 mm
- net /EN_5L: track 2.19 -> 4.67 mm
- net /BTN_USER2: track 56.8 -> 59.1 mm
- net /uSW1: track 416.3 -> 418.7 mm
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