File: Satisfactron_2025.kicad_pcb (KiCad board)
At the start: 2 copper layers, 409.4 x 93 mm, 153 parts, among them J1 USB-TYPE-C-018, J10 GT-BTP30002-0350B-019B, J11 Conn_01x03, J12 LED strip, J2 GT-BTP30002-0350B-019B, J3 TF_PUSH, J4 GT-BTP30002-0350B-019B, J5 PZ254V-11-04P_C2691448, J6 Conn_01x06, J7 GT-BTP30002-0350B-019B, J8 GT-BTP30002-0350B-019B, J9 GT-BTP30002-0350B-019B, Q1 2N7002, SW1 MSK-22D18G4_051, SW10 SPVN310101, SW11 SPVN310101, SW12 SPVN310101, SW13 SPVN310101, SW14 SPVN310101, SW15 SPVN310101, SW2 TS-1088-AR02016, SW3 SPVN310101, SW4 SPVN310101, SW5 TS-1088-AR02016, SW6 TS-1088-AR02016, SW7 TS-1088-AR02016, SW8 SPVN310101, SW9 SPVN310101, U1 AMS1117-3.3, U10 WS2811C, U11 WS2811C, U12 WS2811C, U13 WS2811C, U14 TSSP77038TT, U2 TPS82130, U3 ESP32-S3-WROOM-1-N16R8, U4 TSSP77038TR, U5 TSSP77038TR, U6 TSSP77038TR, U7 TSSP77038TR, U8 TSSP77038TR, U9 WS2811C

Commit message: Minor corrections
Parts:
- added SW16: SPVN310101, Switch_KSL:SW-SMD_SPVN310101, F.Cu at (45.8, 117.7)
- added SW17: SPVN310101, Switch_KSL:SW-SMD_SPVN310101, F.Cu at (45.8, 123.4)
- added SW18: SPVN310101, Switch_KSL:SW-SMD_SPVN310101, F.Cu at (45.8, 129.1)
- added SW19: SPVN310101, Switch_KSL:SW-SMD_SPVN310101, F.Cu at (45.8, 134.8)
- added SW20: SPVN310101, Switch_KSL:SW-SMD_SPVN310101, F.Cu at (45.8, 140.5)
- C11, C22: moved to B.Cu
- moved SW6 4.00 mm to (440.2, 72.8), turned to 90 degrees
Routing:
- net GND: track 1977.7 -> 1982.5 mm
- net /ESP32_EN: track 42.9 -> 44.7 mm
Other:
- board text added: "- +"

Commit message: Routing and zones complete, silkscreen in progress
Parts:
- added G***: LOGO, LOGO, F.Cu at (359.0, 100.5)
- added G***: LOGO, LOGO, F.Cu at (387.0, 100.5)
- added G***: LOGO, LOGO, F.Cu at (380.0, 100.5)
- added G***: LOGO, LOGO, F.Cu at (313.0, 100.5)
- added G***: LOGO, LOGO, F.Cu at (231.0, 100.5)
- added G***: LOGO, LOGO, F.Cu at (157.0, 100.5)
- added G***: LOGO, LOGO, F.Cu at (89.0, 100.5)
- added G***: LOGO, LOGO, F.Cu at (373.0, 100.5)
- added G***: LOGO, LOGO, F.Cu at (306.0, 100.5)
- added G***: LOGO, LOGO, F.Cu at (299.0, 100.5)
- added G***: LOGO, LOGO, F.Cu at (224.0, 100.5)
- added G***: LOGO, LOGO, F.Cu at (366.0, 100.5)
- added G***: LOGO, LOGO, F.Cu at (164.0, 100.5)
- added G***: LOGO, LOGO, F.Cu at (292.0, 100.5)
- added G***: LOGO, LOGO, F.Cu at (238.0, 100.5)
Routing:
- net GND: track 1982.5 -> 1969.9 mm
- net /MISO: track 64.2 -> 65.2 mm
- added copper zone on B.Cu, net GND
- added copper zone on F.Cu, net GND
Other:
- board text added: "Satisfactron"

Commit message: RC last check, silkscreen done
Parts:
- J11: moved to B.Cu
- Q1: footprint Package_TO_SOT_SMD:SOT-23_Handsoldering -> Package_TO_SOT_SMD:SOT-23
- moved Q1 0.10 mm to (418.1, 84.0)
- turned J11 to -90 degrees
- renumbered U14 to U99
Other:
- board text added: "+"
- board text added: "3V3"
- board text added: "Audran CARON"
- board text added: "Authors:"
- board text added: "EN"
- board text added: "G"
- board text added: "RX"
- board text added: "Raphaël CASIMIR"
- board text added: "S"
- board text added: "Source:"
- board text added: "TX"
- board text added: "github.com/jazari-akuna/satisfactron"
- board text added: "h1"

Commit message: Stars are shiny now
Parts:
- removed the G*** at (359.0, 100.5)
- removed the G*** at (387.0, 100.5)
- removed the G*** at (380.0, 100.5)
- removed the G*** at (313.0, 100.5)
- removed the G*** at (231.0, 100.5)
- removed the G*** at (157.0, 100.5)
- removed the G*** at (373.0, 100.5)
- removed the G*** at (306.0, 100.5)
- removed the G*** at (299.0, 100.5)
- removed the G*** at (224.0, 100.5)
- removed the G*** at (366.0, 100.5)
- removed the G*** at (164.0, 100.5)
- removed the G*** at (292.0, 100.5)
- removed the G*** at (238.0, 100.5)
- added G*** (x2): LOGO, LOGO, F.Cu at (306.0, 100.5)
- added G*** (x2): LOGO, LOGO, F.Cu at (380.0, 100.5)
- added G*** (x2): LOGO, LOGO, F.Cu at (299.0, 100.5)
- added G*** (x2): LOGO, LOGO, F.Cu at (387.0, 100.5)
- added G*** (x2): LOGO, LOGO, F.Cu at (359.0, 100.5)
- added G*** (x2): LOGO, LOGO, F.Cu at (231.0, 100.5)
- added G*** (x2): LOGO, LOGO, F.Cu at (157.0, 100.5)
- added G*** (x2): LOGO, LOGO, F.Cu at (224.0, 100.5)
- added G*** (x2): LOGO, LOGO, F.Cu at (366.0, 100.5)
- added G*** (x2): LOGO, LOGO, F.Cu at (238.0, 100.5)
- added G*** (x2): LOGO, LOGO, F.Cu at (164.0, 100.5)
- added G*** (x2): LOGO, LOGO, F.Cu at (373.0, 100.5)
- added G*** (x2): LOGO, LOGO, F.Cu at (313.0, 100.5)
- added G*** (x2): LOGO, LOGO, F.Cu at (292.0, 100.5)
- added G***: LOGO, LOGO, F.Cu at (89.0, 100.5)
Routing:
- net /IRSENS_3: track 268.7 -> 272.2 mm
- net /IRSENS_2: track 341.5 -> 343.4 mm
Other:
- board text added: "JLCJLCJLCJLC"
- board text added: "RESET"

Commit message: Production file (incl. Step)
Routing:
- net /ESP32_EN: track 44.7 -> 42.2 mm
- net /SCK: track 61.7 -> 64.0 mm
- net /MISO: track 65.2 -> 67.2 mm
- net /MOSI: track 60.6 -> 62.2 mm
- net /SERVO1: track 41.9 -> 43.5 mm
Other:
- board size 409.4 x 93 mm -> 409.5 x 93 mm
- board text added: "OFF"
- board text added: "ON"
- board text added: "POWER"
